Commit message: 修复 raxis1_link 惯性值（质量从 0 改为 0.21943 kg）

File: dual_arm_description/urdf/dual_arm_1kg.urdf.xacro (robot description, xacro)
@@ -230,7 +230,7 @@
   <link name="raxis1_link">
     <inertial>
-      <origin xyz="0 0 0" rpy="0 0 0" />
-      <mass value="0" />
-      <inertia ixx="0" ixy="0" ixz="0" iyy="0" iyz="0" izz="0" />
+      <origin xyz="-0.0063819 3.8724E-06 0.0020017" rpy="0 0 0" />
+      <mass value="0.21943" />
+      <inertia ixx="0.00016599" ixy="-2.3484E-07" ixz="2.0611E-07" iyy="0.00012603" iyz="-1.1767E-05" izz="0.0001292" />
     </inertial>
     <visual>

Commit message: 修复了move group中途崩溃的问题，现在可以正常解逆运动学了

File: dual_arm_description/urdf/dual_arm_1kg.urdf.xacro (robot description, xacro)
@@ -21,5 +21,5 @@
       <origin xyz="0 0 0" rpy="0 0 0" />
       <geometry>
-        <mesh filename="package://dual_arm_description/meshes/base_link.STL" />
+        <box size="0.4 0.4 0.2" />
       </geometry>
     </collision>
@@ -43,5 +43,5 @@
       <origin xyz="0 0 0" rpy="0 0 0" />
       <geometry>
-        <mesh filename="package://dual_arm_description/meshes/laxis1_link.STL" />
+        <cylinder length="0.1" radius="0.05" />
       </geometry>
     </collision>
@@ -72,5 +72,5 @@
       <origin xyz="0 0 0" rpy="0 0 0" />
       <geometry>
-        <mesh filename="package://dual_arm_description/meshes/laxis2_link.STL" />
+        <cylinder length="0.1" radius="0.05" />
       </geometry>
     </collision>
@@ -246,5 +246,5 @@
       <origin xyz="0 0 0" rpy="0 0 0" />
       <geometry>
-        <mesh filename="package://dual_arm_description/meshes/raxis1_link.STL" />
+        <cylinder length="0.1" radius="0.05" />
       </geometry>
     </collision>
@@ -275,5 +275,5 @@
       <origin xyz="0 0 0" rpy="0 0 0" />
       <geometry>
-        <mesh filename="package://dual_arm_description/meshes/raxis2_link.STL" />
+        <cylinder length="0.1" radius="0.05" />
       </geometry>
     </collision>

Commit message: 把urdf中的初始位姿与实物同步

File: dual_arm_description/urdf/dual_arm_1kg.urdf.xacro (robot description, xacro)
@@ -41,5 +41,5 @@
     </visual>
     <collision>
-      <origin xyz="0 0 0" rpy="0 0 0" />
+      <origin xyz="0 0 0" rpy="0 1.5708 0" />
       <geometry>
         <cylinder length="0.1" radius="0.05" />
@@ -48,8 +48,8 @@
   </link>
   <joint name="laxis1_joint" type="revolute">
-    <origin xyz="0.12844 -0.010901 0.9108" rpy="2.3441 0 -0.084669" />
+    <origin xyz="0.12844 -0.010901 0.9108" rpy="1.5941 0 -0.084669" />
     <parent link="base_link" />
     <child link="laxis1_link" />
-    <axis xyz="1 0 0" />
+    <axis xyz="-1 0 0" />
     <limit lower="-3.14" upper="3.14" effort="20" velocity="2.0" />
   </joint>
@@ -70,5 +70,5 @@
     </visual>
     <collision>
-      <origin xyz="0 0 0" rpy="0 0 0" />
+      <origin xyz="0 0 0" rpy="0 1.5708 0" />
       <geometry>
         <cylinder length="0.1" radius="0.05" />
@@ -77,5 +77,5 @@
   </link>
   <joint name="laxis2_joint" type="revolute">
-    <origin xyz="0.0774 -3.3783E-05 0.01715" rpy="-1.6846 -1.5688 -1.5708" />
+    <origin xyz="0.0774 -3.3783E-05 0.01715" rpy="-2.8 -1.5688 -1.5708" />
     <parent link="laxis1_link" />
     <child link="laxis2_link" />
@@ -164,5 +164,5 @@
   </link>
   <joint name="laxis5_joint" type="revolute">
-    <origin xyz="0.068269 -0.019 -0.082391" rpy="-2.2242 0.24666 1.8795" />
+    <origin xyz="0.068269 -0.019 -0.082391" rpy="-2.152377 0.398915 2.104409" />
     <parent link="laxis4_link" />
     <child link="laxis5_link" />
@@ -244,5 +244,5 @@
     </visual>
     <collision>
-      <origin xyz="0 0 0" rpy="0 0 0" />
+      <origin xyz="-0.03 0 0" rpy="0 1.5708 0" />
       <geometry>
         <cylinder length="0.1" radius="0.05" />
@@ -251,8 +251,8 @@
   </link>
   <joint name="raxis1_joint" type="revolute">
-    <origin xyz="-0.1541 0.013079 0.9108" rpy="2.2799 0 3.0569" />
+    <origin xyz="-0.1541 0.013079 0.9108" rpy="0.7964 0 3.0569" />
     <parent link="base_link" />
     <child link="raxis1_link" />
-    <axis xyz="1 0 0" />
+    <axis xyz="-1 0 0" />
     <limit lower="-3.14" upper="3.14" effort="20" velocity="2.0" />
   </joint>
@@ -273,5 +273,5 @@
     </visual>
     <collision>
-      <origin xyz="0 0 0" rpy="0 0 0" />
+      <origin xyz="0 0 0" rpy="0 1.5708 0" />
       <geometry>
         <cylinder length="0.1" radius="0.05" />
@@ -280,8 +280,8 @@
   </link>
   <joint name="raxis2_joint" type="revolute">
-    <origin xyz="0.051649 -0.012151 0.012103" rpy="-1.6846 -0.78343 -1.5708" />
+    <origin xyz="0.051649 -0.012151 0.012103" rpy="-2.8016 -0.78343 -1.5708" />
     <parent link="raxis1_link" />
     <child link="raxis2_link" />
-    <axis xyz="1 0 0" />
+    <axis xyz="-1 0 0" />
     <limit lower="-3.14" upper="3.14" effort="20" velocity="2.0" />
   </joint>
@@ -367,5 +367,5 @@
   </link>
   <joint name="raxis5_joint" type="revolute">
-    <origin xyz="0.068269 -0.019 -0.082391" rpy="-2.2242 0.24666 1.8795" />
+    <origin xyz="0.068269 -0.019 -0.082391" rpy="-0.995458 -0.408458 -1.021292" />
     <parent link="raxis4_link" />
     <child link="raxis5_link" />
@@ -440,5 +440,7 @@
       <command_interface name="position"/>
       <command_interface name="velocity"/>
-      <state_interface name="position"/>
+      <state_interface name="position">
+        <param name="initial_value">0.0</param>
+      </state_interface>
       <state_interface name="velocity"/>
       <state_interface name="effort"/>
@@ -447,5 +449,7 @@
       <command_interface name="position"/>
       <command_interface name="velocity"/>
-      <state_interface name="position"/>
+      <state_interface name="position">
+        <param name="initial_value">0.0</param>
+      </state_interface>
       <state_interface name="velocity"/>
       <state_interface name="effort"/>
@@ -454,5 +458,7 @@
       <command_interface name="position"/>
       <command_interface name="velocity"/>
-      <state_interface name="position"/>
+      <state_interface name="position">
+        <param name="initial_value">0.0</param>
+      </state_interface>
       <state_interface name="velocity"/>
       <state_interface name="effort"/>
@@ -461,5 +467,7 @@
       <command_interface name="position"/>
       <command_interface name="velocity"/>
-      <state_interface name="position"/>
+      <state_interface name="position">
+        <param name="initial_value">0.0</param>
+      </state_interface>
       <state_interface name="velocity"/>
       <state_interface name="effort"/>
@@ -468,5 +476,7 @@
       <command_interface name="position"/>
       <command_interface name="velocity"/>
-      <state_interface name="position"/>
+      <state_interface name="position">
+        <param name="initial_value">0.0</param>
+      </state_interface>
       <state_interface name="velocity"/>
       <state_interface name="effort"/>
@@ -475,5 +485,7 @@
       <command_interface name="position"/>
       <command_interface name="velocity"/>
-      <state_interface name="position"/>
+      <state_interface name="position">
+        <param name="initial_value">0.0</param>
+      </state_interface>
       <state_interface name="velocity"/>
       <state_interface name="effort"/>
@@ -482,5 +494,7 @@
       <command_interface name="position"/>
       <command_interface name="velocity"/>
-      <state_interface name="position"/>
+      <state_interface name="position">
+        <param name="initial_value">0.0</param>
+      </state_interface>
       <state_interface name="velocity"/>
       <state_interface name="effort"/>
@@ -490,5 +504,7 @@
       <command_interface name="position"/>
       <command_interface name="velocity"/>
-      <state_interface name="position"/>
+      <state_interface name="position">
+        <param name="initial_value">0.0</param>
+      </state_interface>
       <state_interface name="velocity"/>
       <state_interface name="effort"/>
@@ -497,5 +513,7 @@
       <command_interface name="position"/>
       <command_interface name="velocity"/>
-      <state_interface name="position"/>
+      <state_interface name="position">
+        <param name="initial_value">0.0</param>
+      </state_interface>
       <state_interface name="velocity"/>
       <state_interface name="effort"/>
@@ -504,5 +522,7 @@
       <command_interface name="position"/>
       <command_interface name="velocity"/>
-      <state_interface name="position"/>
+      <state_interface name="position">
+        <param name="initial_value">0.0</param>
+      </state_interface>
       <state_interface name="velocity"/>
       <state_interface name="effort"/>
@@ -511,5 +531,7 @@
       <command_interface name="position"/>
       <command_interface name="velocity"/>
-      <state_interface name="position"/>
+      <state_interface name="position">
+        <param name="initial_value">0.0</param>
+      </state_interface>
       <state_interface name="velocity"/>
       <state_interface name="effort"/>
@@ -518,5 +540,7 @@
       <command_interface name="position"/>
       <command_interface name="velocity"/>
-      <state_interface name="position"/>
+      <state_interface name="position">
+        <param name="initial_value">0.0</param>
+      </state_interface>
       <state_interface name="velocity"/>
       <state_interface name="effort"/>
@@ -525,5 +549,7 @@
       <command_interface name="position"/>
       <command_interface name="velocity"/>
-      <state_interface name="position"/>
+      <state_interface name="position">
+        <param name="initial_value">0.0</param>
+      </state_interface>
       <state_interface name="velocity"/>
       <state_interface name="effort"/>
@@ -532,5 +558,7 @@
       <command_interface name="position"/>
       <command_interface name="velocity"/>
-      <state_interface name="position"/>
+      <state_interface name="position">
+        <param name="initial_value">0.0</param>
+      </state_interface>
       <state_interface name="velocity"/>
       <state_interface name="effort"/>

Commit message: 修复了execute后电机乱转的问题

File: dual_arm_description/urdf/dual_arm_1kg.urdf.xacro (robot description, xacro)
@@ -51,5 +51,5 @@
     <parent link="base_link" />
     <child link="laxis1_link" />
-    <axis xyz="-1 0 0" />
+    <axis xyz="1 0 0" />
     <limit lower="-3.14" upper="3.14" effort="20" velocity="2.0" />
   </joint>
@@ -106,5 +106,5 @@
   </link>
   <joint name="laxis3_joint" type="revolute">
-    <origin xyz="-0.016833 0.034747 0.1012" rpy="1.748 -0.28299 -2.1411" />
+    <origin xyz="-0.016833 0.034747 0.1012" rpy="1.393593 0.282990 1.000493" />
     <parent link="laxis2_link" />
     <child link="laxis3_link" />
@@ -164,5 +164,5 @@
   </link>
   <joint name="laxis5_joint" type="revolute">
-    <origin xyz="0.068269 -0.019 -0.082391" rpy="-2.152377 0.398915 2.104409" />
+    <origin xyz="0.068269 -0.019 -0.082391" rpy="-0.989216 -0.398915 -1.037184" />
     <parent link="laxis4_link" />
     <child link="laxis5_link" />
@@ -254,5 +254,5 @@
     <parent link="base_link" />
     <child link="raxis1_link" />
-    <axis xyz="-1 0 0" />
+    <axis xyz="1 0 0" />
     <limit lower="-3.14" upper="3.14" effort="20" velocity="2.0" />
   </joint>

Commit message: 优化了实物实验

File: dual_arm_description/urdf/dual_arm_1kg.urdf.xacro (robot description, xacro)
@@ -41,7 +41,7 @@
     </visual>
     <collision>
-      <origin xyz="0 0 0" rpy="0 1.5708 0" />
-      <geometry>
-        <cylinder length="0.1" radius="0.05" />
+      <origin xyz="-0.015 0 0" rpy="0 1.5708 0" />
+      <geometry>
+        <cylinder length="0.08" radius="0.04" />
       </geometry>
     </collision>
@@ -72,5 +72,5 @@
       <origin xyz="0 0 0" rpy="0 1.5708 0" />
       <geometry>
-        <cylinder length="0.1" radius="0.05" />
+        <cylinder length="0.08" radius="0.04" />
       </geometry>
     </collision>
